Commit message: third commit

File: urdf/macros.xacro (robot description, xacro)
@@ -13,15 +13,15 @@
     <collision name="collision_chassis">
       <geometry>
-        <!--<box size="0.5 0.3 0.07"/>-->
-        <mesh filename="package://amr_2wr/models/amr_2wr/meshes/Chasis.stl" scale="0.001 0.001 0.001"/>
+        <box size="0.5 0.3 0.07"/>
+        <!--<mesh filename="package://amr_2wr/models/amr_2wr/meshes/Chasis.stl" scale="0.001 0.001 0.001"/>-->
       </geometry>
     </collision>
     <visual>
-      <origin rpy="0 0 0" xyz="0 0 0"/>
+      <origin rpy="0 0 -1.5707" xyz="0.075 -0.055 -0.1"/>
       <geometry>
         <!--<box size="0.5 0.3 0.07"/>-->
-        <mesh filename="package://amr_2wr/models/amr_2wr/meshes/Chasis.stl" scale="0.001 0.001 0.001"/>
+        <mesh filename="package://amr_2wr/models/amr_2wr/meshes/Chasis.stl" scale="0.00185 0.00185 0.00185" />
       </geometry>
-      <material name="blue"/>
+      <material name="red"/>
     </visual>
     <!-- caster front -->
@@ -45,5 +45,5 @@
       <origin rpy=" 0 0 0" xyz="0.2 0 -0.05"/>
       <geometry>
-        <sphere radius="0.05"/>
+        <sphere radius="0.001"/>
       </geometry>
     </visual>
@@ -60,13 +60,14 @@
       	<origin rpy="0 1.5707 1.5707" xyz="0 0 0"/>
       	<geometry>
-        <!--<cylinder length="0.04" radius="0.1"/>-->
-        <mesh filename="package://amr_2wr/models/amr_2wr/meshes/Wheel.stl" scale="0.001 0.001 0.001"/>
+        <cylinder length="0.04" radius="0.1"/>
+        <!--<mesh filename="package://amr_2wr/models/amr_2wr/meshes/Wheel.stl" scale="0.001 0.001 0.001"/>-->
       	</geometry>
     	</collision>
     	<visual name="${link_name}_visual">
-      	<origin rpy="0 1.5707 1.5707" xyz="0 0 0"/>
+    	<!-- ONLY CHANGE XYZ -->
+      	<origin rpy="0 0 1.5707" xyz="0 0 0"/>
       	<geometry>
         <!--<cylinder length="0.04" radius="0.1"/>-->
-        <mesh filename="package://amr_2wr/models/amr_2wr/meshes/Wheel.stl" scale="0.001 0.001 0.001"/>
+        <mesh filename="package://amr_2wr/models/amr_2wr/meshes/Wheel.stl" scale="0.00185 0.00185 0.00185"/>
       	</geometry>
     	</visual>
@@ -93,9 +94,10 @@
     </inertial>
     <visual>
-        <origin xyz="0 0 0" rpy="0 0 0" />
+        <origin xyz="0.155 -0.45 -0.11" rpy="0 0 -1.5707"/>
         <geometry>
-        <cylinder radius="0.05" length="0.1"/>
+        <!--<cylinder radius="0.05" length="0.1"/>-->
+        <mesh filename="package://amr_2wr/models/amr_2wr/meshes/RpLidar.stl" scale="0.00185 0.00185 0.00185" />
         </geometry>
-        <material name="white" />
+        <material name="black" />
     </visual>
     <collision>

Commit message: fourth commit

File: urdf/macros.xacro (robot description, xacro)
@@ -60,11 +60,12 @@
       	<origin rpy="0 1.5707 1.5707" xyz="0 0 0"/>
       	<geometry>
-        <cylinder length="0.04" radius="0.1"/>
-        <!--<mesh filename="package://amr_2wr/models/amr_2wr/meshes/Wheel.stl" scale="0.001 0.001 0.001"/>-->
+        <!--<cylinder length="0.04" radius="0.1"/>-->
+        <mesh filename="package://amr_2wr/models/amr_2wr/meshes/Wheel.stl" scale="0.00185 0.00185 0.00185"/>
       	</geometry>
     	</collision>
     	<visual name="${link_name}_visual">
     	<!-- ONLY CHANGE XYZ -->
-      	<origin rpy="0 0 1.5707" xyz="0 0 0"/>
+    	<!--<origin rpy="0 1.5707 1.5707" xyz="0 0 0"/>-->
+      	<!--<origin rpy="0 0 1.5707" xyz="-0.1 0.225 -0.085"/>-->
       	<geometry>
         <!--<cylinder length="0.04" radius="0.1"/>-->
