Commit message: second commit

File: urdf/amr_2wr.xacro (robot description, xacro)
@@ -1,115 +1,12 @@
-<?xml version="1.0"?>
-<robot name="amr_2wr" xmlns:xacro="http://ros.org/wiki/xacro">
-    <material name="blue">
-	    <color rgba="0 0 0.8 1"/>
-    </material>
-    <material name="white">
-	    <color rgba="1 1 1 1"/>
-    </material>
-    <material name="black">
-	    <color rgba="0 0 0 1"/>
-    </material>
-    <material name="green">
-        <color rgba="0.0 0.8 0.0 1.0"/>
-    </material>
-    <link name="base_link">
-        <!--<visual>
-          <geometry>
-             <box size="0.24 0.24 0.001"/>
-          </geometry>
-          <material name="white"/>
-          <origin rpy="0 0 0" xyz="0 0 0.0005"/>
-          <material>
-            <color rgba="0 0 0.8 1" />
-          </material>
-        </visual> -->
-        <collision>
-          <origin rpy="0 0 0" xyz="0 0 0.0005"/>
-          <geometry>
-            <box size="0.22 0.22 0.001"/>
-          </geometry>
-        </collision>
-    </link>
-    <joint name="base_link_joint" type="fixed">
-        <origin xyz="0 0 0.026" rpy="0 0 -1.5708" />
-        <parent link="base_link" />
-        <child link="base_plate" />
-    </joint>
-    <link name="base_plate">
-    <visual>
-      <origin rpy="0 0 0" xyz="0.03 0 -0.026"/>
-      <geometry>
-        <mesh filename="package://amr_2wr/models/amr_2wr/meshes/Chasis.stl" scale="0.001 0.001 0.001"/>
-      </geometry>
-      <material name="white"/>
-    </visual>
-    <collision>
-      <origin rpy="0 0 0" xyz="0.03 0 -0.026"  />
-      <geometry>
-        <mesh filename="package://amr_2wr/models/amr_2wr/meshes/Chasis.stl" scale="0.001 0.001 0.001" />
-      </geometry>
-    </collision>
-    </link>
-    <joint name="right_wheel_joint" type="continuous">
-        <origin xyz="-0.08 -0.06 0.015" rpy="0 0 0" />
-        <parent link="base_plate" />
-        <child link="right_wheel" />
-        <axis xyz="-1 0 0" />
-    </joint>
-    <link name="right_wheel">
-    <visual>
-      <origin rpy="0 0 0" xyz="0.11 0.059 -0.04"/>
-      <geometry>
-        <mesh filename="package://amr_2wr/models/amr_2wr/meshes/Wheel.stl" scale="0.001 0.001 0.001"/>
-      </geometry>
-      <material name="black"/>
-    </visual>
-    <collision>
-      <origin rpy="0 0 0" xyz="0.11 0.059 -0.04"/>
-      <geometry>
-        <mesh filename="package://amr_2wr/models/amr_2wr/meshes/Wheel.stl" scale="0.001 0.001 0.001" />
-      </geometry>
-    </collision>
-    </link>
-    <joint name="left_wheel_joint" type="continuous">
-        <origin xyz="0.08 -0.06 0.015" rpy="0 0 0" />
-        <parent link="base_plate" />
-        <child link="left_wheel" />
-        <axis xyz="-1 0 0" />
-    </joint>
-    <link name="left_wheel">
-    <visual>
-      <origin rpy="0 0 0" xyz="0.133 0.059 -0.04"/>
-      <geometry>
-        <mesh filename="package://amr_2wr/models/amr_2wr/meshes/Wheel.stl" scale="0.001 0.001 0.001"/>
-      </geometry>
-      <material name="black"/>
-    </visual>
-    <collision>
-      <origin rpy="0 0 0" xyz="0.133 0.059 -0.04"/>
-      <geometry>
-        <mesh filename="package://amr_2wr/models/amr_2wr/meshes/Wheel.stl" scale="0.001 0.001 0.001" />
-      </geometry>
-    </collision>
-    </link>
-    <joint name="laser_joint" type="fixed">
-        <origin xyz="0 0.040 0.090" rpy="0 0 1.5708" />
-        <parent link="base_plate" />
-        <child link="laser" />
-    </joint>
-    <link name="laser">
-    <visual>
-      <origin rpy="0 0 -1.5708" xyz="0.084 -0.242 -0.098"/>
-      <geometry>
-        <mesh filename="package://amr_2wr/models/amr_2wr/meshes/RpLidar.stl" scale="0.001 0.001 0.001"/>
-      </geometry>
-      <material name="blue"/>
-    </visual>
-    <collision>
-      <origin rpy="0 0 0" xyz="0.242 0.084 -0.098"  />
-      <geometry>
-        <mesh filename="package://amr_2wr/models/amr_2wr/meshes/RpLidar.stl" scale="0.001 0.001 0.001" />
-      </geometry>
-    </collision>
-    </link>
+<?xml version="1.0" ?>
+<robot name="amr_2wr" xmlns:xacro="http://www.ros.org/wiki/xacro">
+  <xacro:include filename="$(find amr_2wr)/urdf/materials.xacro"/>
+  <xacro:include filename="$(find amr_2wr)/urdf/amr_2wr.gazebo"/>
+  <xacro:include filename="$(find amr_2wr)/urdf/macros.xacro"/>
+  <xacro:chassis/>
+  <xacro:lidar mass="1" r="0.05" l="0.1"/>
+  <xacro:link_wheel link_name="link_right_wheel"/>
+  <xacro:wheel_joint position="right" x="-0.05" y="0.15" z="0" child="link_right_wheel"/>
+  <xacro:link_wheel link_name="link_left_wheel"/>
+  <xacro:wheel_joint position="left" x="-0.05" y="-0.15" z="0" child="link_left_wheel"/>
 </robot>

Commit message: fifth commit

File: urdf/amr_2wr.xacro (robot description, xacro)
@@ -7,6 +7,6 @@
   <xacro:lidar mass="1" r="0.05" l="0.1"/>
   <xacro:link_wheel link_name="link_right_wheel"/>
-  <xacro:wheel_joint position="right" x="-0.05" y="0.15" z="0" child="link_right_wheel"/>
+  <xacro:wheel_joint position="right" x="-0.05" y="-0.15" z="0" child="link_right_wheel"/>
   <xacro:link_wheel link_name="link_left_wheel"/>
-  <xacro:wheel_joint position="left" x="-0.05" y="-0.15" z="0" child="link_left_wheel"/>
+  <xacro:wheel_joint position="left" x="-0.05" y="0.15" z="0" child="link_left_wheel"/>
 </robot>

File: urdf/macros.xacro (robot description, xacro)
@@ -53,5 +53,5 @@
 	<link name="${link_name}">
     	<inertial>
-      	<mass value="0.2"/>
+      	<mass value="0.5"/>
       	<origin rpy="0 1.5707 1.5707" xyz="0 0 0"/>
       	<inertia ixx="0.000526666666667" ixy="0" ixz="0" iyy="0.000526666666667" iyz="0" izz="0.001"/>
@@ -60,16 +60,18 @@
       	<origin rpy="0 1.5707 1.5707" xyz="0 0 0"/>
       	<geometry>
-        <!--<cylinder length="0.04" radius="0.1"/>-->
-        <mesh filename="package://amr_2wr/models/amr_2wr/meshes/Wheel.stl" scale="0.00185 0.00185 0.00185"/>
+        <cylinder length="0.04" radius="0.1"/>
+        <!--<mesh filename="package://amr_2wr/models/amr_2wr/meshes/Wheel.stl" scale="0.00185 0.00185 0.00185"/>-->
       	</geometry>
     	</collision>
     	<visual name="${link_name}_visual">
     	<!-- ONLY CHANGE XYZ -->
-    	<!--<origin rpy="0 1.5707 1.5707" xyz="0 0 0"/>-->
+    	<origin rpy="0 1.5707 1.5707" xyz="0 -0.02 0"/>
       	<!--<origin rpy="0 0 1.5707" xyz="-0.1 0.225 -0.085"/>-->
+      	<!--<origin rpy="0 0 -1.57 07" xyz="0.084 -0.242 -0.098"/>-->
       	<geometry>
         <!--<cylinder length="0.04" radius="0.1"/>-->
         <mesh filename="package://amr_2wr/models/amr_2wr/meshes/Wheel.stl" scale="0.00185 0.00185 0.00185"/>
       	</geometry>
+      	<material name="black"/>
     	</visual>
 	</link>
